File: Hardware/Sparkfun_AS6212_Qwiic.sch (EAGLE design)
At the start: 30 parts, among them J1 PTH, J2 QWIIC_RA, J3 QWIIC_RA, U2 AS6212

Commit message: Layout ready for review
Parts:
- removed JP6: JUMPER-SMT_3_1-NC_TRACE_NO-SILK, SparkFun-Jumpers:JUMPER-SMT_3_1-NC_TRACE_NO-SILK
- removed JP7: JUMPER-SMT_3_NO_NO_SILK, SparkFun-Jumpers:JUMPER-SMT_3_NO_NO_SILK
- added JP10: JUMPER-SMT_3_1-NC_TRACE_NO-SILK, SparkFun-Jumpers:JUMPER-SMT_3_1-NC_TRACE_NO-SILK
- added JP11: JUMPER-SMT_3_NO_NO_SILK, SparkFun-Jumpers:JUMPER-SMT_3_NO_NO_SILK
Connections:
- net ALERT/ADD1: now also JP10.2, JP11.2; no longer JP6.2, JP7.2
- net GND: now also JP11.3; no longer JP6.3
- net N$5: now also JP10.3; no longer JP7.1
- net SCL: now also JP10.1; no longer JP7.3
- net SDA: now also JP11.1; no longer JP6.1
Other:
- note added: "0x44"
- note added: "0x45"
- note added: "0x46"
- note added: "0x47"
- note added: "ADD0"
- note added: "ALERT/ ADD1"
- note added: "Alert Functionality Enabled"
- note added: "No"
- note added: "There are 8 jumper selectable I2C addresses DEFAULT: 0x48 (Alert Functionality Enabled)"
- note added: "VCC (PU)"
- note added: "Yes"
- note removed: "I2C Address select"
- note removed: "There are 12 jumper selectable I2C addresses DEFAULT: 0x48"
- moved on the sheet: JP4, JP5, R2, R6

Commit message: design review group
-adjusted some traces and added more GND vias for return currents
-changed to 3V3 on label to avoid dot not printing nice
-GND symbols updated to new libraries
Parts:
- JP2, JP3, JP8, JP9: device SparkFun:STAND-OFF -> SparkFun-Hardware:STAND-OFF
Changed lines of the file:
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@@
 <layer number="56" name="wert" color="7" fill="1" visible="no" active="no"/>
 <layer number="57" name="tCAD" color="7" fill="1" visible="no" active="no"/>
+<layer number="58" name="bCAD" color="7" fill="1" visible="no" active="no"/>
 <layer number="59" name="tCarbon" color="7" fill="1" visible="no" active="no"/>
 <layer number="60" name="bCarbon" color="7" fill="1" visible="no" active="no"/>
@@
 <layer number="250" name="Descript" color="3" fill="1" visible="no" active="no"/>
 <layer number="251" name="SMDround" color="12" fill="11" visible="no" active="no"/>
+<layer number="253" name="Extra" color="7" fill="1" visible="no" active="no"/>
 <layer number="254" name="cooling" color="7" fill="1" visible="yes" active="yes"/>
 <layer number="255" name="routoute" color="7" fill="1" visible="yes" active="yes"/>
@@
 <part name="SUPPLY3" library="SparkFun-PowerSymbols" deviceset="3.3V" device=""/>
 <part name="SUPPLY4" library="SparkFun-PowerSymbols" deviceset="3.3V" device=""/>
-<part name="GND7" library="SparkFun" deviceset="GND" device=""/>
-<part name="GND5" library="SparkFun" deviceset="GND" device=""/>
-<part name="GND6" library="SparkFun" deviceset="GND" device=""/>
+<part name="GND7" library="SparkFun-PowerSymbols" deviceset="GND" device=""/>
+<part name="GND5" library="SparkFun-PowerSymbols" deviceset="GND" device=""/>
+<part name="GND6" library="SparkFun-PowerSymbols" deviceset="GND" device=""/>
 <part name="SUPPLY5" library="SparkFun-PowerSymbols" library_urn="urn:adsk.eagle:library:530" deviceset="3.3V" device=""/>
 <part name="R2" library="SparkFun-Resistors" deviceset="10KOHM" device="-0603-1/10W-1%" value="10k"/>
@@
 <part name="SUPPLY9" library="SparkFun-PowerSymbols" library_urn="urn:adsk.eagle:library:530" deviceset="3.3V" device=""/>
 <part name="J2" library="SparkFun-Connectors" deviceset="QWIIC_CONNECTOR" device="JS-1MM" value="QWIIC_RA"/>
-<part name="JP8" library="SparkFun" deviceset="STAND-OFF" device=""/>
-<part name="JP9" library="SparkFun" deviceset="STAND-OFF" device=""/>
+<part name="JP8" library="SparkFun-Hardware" deviceset="STAND-OFF" device=""/>
+<part name="JP9" library="SparkFun-Hardware" deviceset="STAND-OFF" device=""/>
 <part name="I2C" library="SparkFun-Jumpers" deviceset="JUMPER-SMT_3_2-NC_TRACE" device="_SILK" package3d_urn="urn:adsk.eagle:package:39289/1" value=""/>
 <part name="JP4" library="SparkFun-Jumpers" deviceset="JUMPER-SMT_3_1-NC_TRACE" device="_NO-SILK" package3d_urn="urn:adsk.eagle:package:39287/1"/>
@@
 <part name="SUPPLY10" library="SparkFun-PowerSymbols" library_urn="urn:adsk.eagle:library:530" deviceset="3.3V" device=""/>
 <part name="JP1" library="SparkFun-Jumpers" deviceset="JUMPER-SMT_2_NC_TRACE" device="_SILK" package3d_urn="urn:adsk.eagle:package:39281/1" value="LED"/>
-<part name="JP2" library="SparkFun" deviceset="STAND-OFF" device=""/>
-<part name="JP3" library="SparkFun" deviceset="STAND-OFF" device=""/>
+<part name="JP2" library="SparkFun-Hardware" deviceset="STAND-OFF" device=""/>
+<part name="JP3" library="SparkFun-Hardware" deviceset="STAND-OFF" device=""/>
 <part name="LOGO4" library="SparkFun-Aesthetics" deviceset="SFE_LOGO_NAME_FLAME" device=".1_INCH"/>
 <part name="FD1" library="SparkFun-Aesthetics" library_urn="urn:adsk.eagle:library:507" deviceset="FIDUCIAL" device="UFIDUCIAL" package3d_urn="urn:adsk.eagle:package:37111/1"/>
